File: _autosave-pilulith.kicad_pcb (KiCad board)
At the start: 6 copper layers, 22.1 x 22.1 mm, 91 parts, among them J101 Conn_01x03_Pin, J103 Conn_ARM_JTAG_SWD_10, Q1 SBC847, SW1 KMT221NG, SW2 KMT221NG, U1 NRF54L15-QFAA-R, U10 LIS2DH, U102 WLA.04, U103 ATECC608B-MAHDA, U104 LF21115TMR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

Commit message: Modified to use nRF54L15 and DFN instead of BGA nRF52. Moving parts to match
Parts:
- added SW3: KMT221NG, Button_Switch_SMD:SW_Push_1P1T_NO_CK_KMR2, B.Cu at (165.9, 110.3)
- moved SW1 12.7 mm to (150.5, 104.0), turned to 90 degrees
- moved J101 10.6 mm to (158.6, 96.2), turned to 0 degrees
- moved Q1 7.13 mm to (154.8, 111.6), turned to -120 degrees
- moved SW2 6.70 mm to (165.5, 97.6), turned to 135 degrees
- moved D3 6.52 mm to (161.4, 112.1), turned to -90 degrees
- moved C102 4.67 mm to (165.4, 110.3), turned to -45 degrees
- moved U106 4.42 mm to (167.6, 106.2), turned to 75 degrees
- moved R106 3.73 mm to (161.0, 114.5), turned to 180 degrees
- moved R104 1.86 mm to (167.8, 109.0)
- moved R103 0.33 mm to (168.7, 103.5), turned to -165 degrees
- turned BT101 to 0 degrees
Routing:
- net Net-(U1-P1.00/XL1): track 0.00 -> 0.22 mm, vias 0 -> 1
