File: phial.kicad_pcb (KiCad board)
At the start: 6 copper layers, 22.1 x 22.1 mm, 100 parts, among them J101 Conn_01x03_Pin, J103 Conn_ARM_JTAG_SWD_10, Q1 SBC847, SW1 KMT221NG, SW2 KMT221NG, SW3 KMT221NG, SW4 KMT221NG, U1 NRF54L15-QFAA-R, U10 LIS2DH, U102 WLA.04, U103 ATECC608B-MAHDA, U104 LF21115TMR, U105 BME280, U106 MP34DT05TR-A, U2 NPM2100-CAAA-R, Y101 32MHz, Y102 32.768K

Commit message: OSHW release prep: docs, license, project rename (pilulith -> phial)
Parts:
- BT101: footprint pilulith:BAT_112TR -> phial:BAT_112TR
- G***: footprint pilulith:pilulith_10mm -> phial:pilulith_10mm
- J101: footprint pilulith:Cabling -> phial:Cabling
- LS1: footprint pilulith:RDTE-4.000-3030-NS1 -> phial:RDTE-4.000-3030-NS1
- SW1, SW2, SW3: footprint pilulith:KMT221NG -> phial:KMT221NG
- SW4: footprint pilulith:SW_EVP-AWED4A -> phial:SW_EVP-AWED4A
- U1: footprint pilulith:QFN40P600X600X90-49N -> phial:QFN40P600X600X90-49N
- U2: footprint pilulith:BGA16N44P4X4_189X191X52N -> phial:BGA16N44P4X4_189X191X52N
